File: pcb/stream_deck_hardware/stream_deck_hardware.sch (KiCad schematic (older format))
At the start: 29 parts, among them J1 Conn_01x03_Female, SW1 SW_Push_LED, SW10 SW_Push_LED, SW11 SW_Push_LED, SW2 Rotary_Encoder_Switch, SW3 SW_Push_LED, SW4 Rotary_Encoder_Switch, SW5 SW_Push_LED, SW6 SW_Push_LED, SW7 Rotary_Encoder_Switch, SW8 SW_Push_LED, SW9 SW_Push_LED

Commit message: electrical schematic desiging
Parts:
- removed D1, D2, D3, D4, D5, D6, D7, D8: WS2812B, LED_SMD:LED_WS2812B_PLCC4_5.0x5.0mm_P3.2mm, symbol LED:WS2812B
- removed J1: Conn_01x03_Female, symbol Connector:Conn_01x03_Female
- removed R1, R2, R3, R4, R5, R6, R7, R8, R9: R, symbol Device:R
- removed SW1, SW10, SW11, SW3, SW5, SW6, SW8, SW9: SW_Push_LED, Button_Switch_Keyboard:SW_Cherry_MX_1.00u_PCB, symbol Switch:SW_Push_LED
- removed SW2, SW4, SW7: Rotary_Encoder_Switch, symbol Device:Rotary_Encoder_Switch
- added U?: STM32F401RCTx, Package_QFP:LQFP-64_10x10mm_P0.5mm, symbol MCU_ST_STM32F4:STM32F401RCTx
Connections:
- net labels removed: +5V, Button_1, GND
- wire segments 75 -> 0
