File: pcb/switches.sch (KiCad schematic (older format))
At the start: 54 parts, among them J5 Conn_01x05_Male, SW1 SW_Push1, SW2 SW_Push2, SW3 SW_Push3, SW4 SW_Push, SW5 SW_Push, SW6 SW_Push, SW7 SW_Push, SW8 SW_Push, SW9 SW_Push

Commit message: Change connectors footprints
Parts:
- removed J5: Conn_01x05_Male, Connector_PinHeader_2.54mm:PinHeader_1x05_P2.54mm_Horizontal, symbol Connector:Conn_01x05_Male
- added J10, J9: GND, TestPoint:TestPoint_Pad_D2.0mm, symbol Connector:Conn_01x01_Female
- added J6: ENC A, TestPoint:TestPoint_Pad_D2.0mm, symbol Connector:Conn_01x01_Female
- added J7: ENC B, TestPoint:TestPoint_Pad_D2.0mm, symbol Connector:Conn_01x01_Female
- added J8: BUTTON, TestPoint:TestPoint_Pad_D2.0mm, symbol Connector:Conn_01x01_Female
Connections:
- net ENC_01_A: now also J7.1 (Pin_1)
- net ENC_01_B: now also J6.1 (Pin_1)
- net GND: now also J10.1 (Pin_1), J9.1 (Pin_1)
- net at C22.1, R33.2, R36.1: now also J8.1 (Pin_1)
Changed lines of the file:
@@
 Wire Wire Line
 	3200 5500 3200 5450
-Connection ~ 3200 5450
 Wire Wire Line
 	3200 5450 3200 5400
@@
 	1    0    0    -1
 $EndComp
-$Comp
-L Connector:Conn_01x05_Male J5
-U 1 1 61E13F1C
-P 2450 5740
-F 0 "J5" H 2090 5840 50  0000 C CNN
-F 1 "Conn_01x05_Male" H 2080 5740 50  0000 C CNN
-F 2 "Connector_PinHeader_2.54mm:PinHeader_1x05_P2.54mm_Horizontal" H 2450 5740 50  0001 C CNN
-F 3 "~" H 2450 5740 50  0001 C CNN
-	1    2450 5740
-	1    0    0    -1
-$EndComp
 Wire Wire Line
 	2650 5840 2780 5840
@@
 	1    0    0    -1
 $EndComp
+Connection ~ 3200 5450
+$Comp
+L Connector:Conn_01x01_Female J?
+U 1 1 61ED4421
+P 2450 5540
+AR Path="/61ED4421" Ref="J?"  Part="1"
+AR Path="/61B99CE8/61ED4421" Ref="J6"  Part="1"
+F 0 "J6" H 2910 5540 50  0000 C CNN
+F 1 "ENC A" H 2590 5540 50  0000 C CNN
+F 2 "TestPoint:TestPoint_Pad_D2.0mm" H 2450 5540 50  0001 C CNN
+F 3 "~" H 2450 5540 50  0001 C CNN
+	1    2450 5540
+	-1   0    0    1
+$EndComp
+$Comp
+L Connector:Conn_01x01_Female J?
+U 1 1 61ED4427
+P 2450 5640
+AR Path="/61ED4427" Ref="J?"  Part="1"
+AR Path="/61B99CE8/61ED4427" Ref="J7"  Part="1"
+F 0 "J7" H 2910 5640 50  0000 C CNN
+F 1 "ENC B" H 2590 5640 50  0000 C CNN
+F 2 "TestPoint:TestPoint_Pad_D2.0mm" H 2450 5640 50  0001 C CNN
+F 3 "~" H 2450 5640 50  0001 C CNN
+	1    2450 5640
+	-1   0    0    1
+$EndComp
+$Comp
+L Connector:Conn_01x01_Female J?
+U 1 1 61ED442D
+P 2450 5740
+AR Path="/61ED442D" Ref="J?"  Part="1"
+AR Path="/61B99CE8/61ED442D" Ref="J8"  Part="1"
+F 0 "J8" H 2910 5740 50  0000 C CNN
+F 1 "BUTTON" H 2610 5740 50  0000 C CNN
+F 2 "TestPoint:TestPoint_Pad_D2.0mm" H 2450 5740 50  0001 C CNN
+F 3 "~" H 2450 5740 50  0001 C CNN
+	1    2450 5740
+	-1   0    0    1
+$EndComp
+$Comp
+L Connector:Conn_01x01_Female J?
+U 1 1 61ED4433
+P 2450 5840
+AR Path="/61ED4433" Ref="J?"  Part="1"
+AR Path="/61B99CE8/61ED4433" Ref="J9"  Part="1"
+F 0 "J9" H 2910 5840 50  0000 C CNN
+F 1 "GND" H 2550 5840 50  0000 C CNN
+F 2 "TestPoint:TestPoint_Pad_D2.0mm" H 2450 5840 50  0001 C CNN
+F 3 "~" H 2450 5840 50  0001 C CNN
+	1    2450 5840
+	-1   0    0    1
+$EndComp
+$Comp
+L Connector:Conn_01x01_Female J?
+U 1 1 61EDA8FA
+P 2450 5940
+AR Path="/61EDA8FA" Ref="J?"  Part="1"
+AR Path="/61B99CE8/61EDA8FA" Ref="J10"  Part="1"
+F 0 "J10" H 2910 5940 50  0000 C CNN
+F 1 "GND" H 2550 5940 50  0000 C CNN
+F 2 "TestPoint:TestPoint_Pad_D2.0mm" H 2450 5940 50  0001 C CNN
+F 3 "~" H 2450 5940 50  0001 C CNN
+	1    2450 5940
+	-1   0    0    1
+$EndComp
 $EndSCHEMATC
