File: pcb/stream_deck_hardware.sch (KiCad schematic (older format))
At the start: 44 parts, among them J1 USB_C_Receptacle_USB2.0, U1 LF33_TO252, U2 STM32F401RCTx, U3 74LVC1G332, U4 AT24CS02-STUM, U5 AT24CS02-STUM, Y1 Crystal_Small

Commit message: COMPONENT PLACEMENT
Parts:
- D1, D2, D3: renamed from D?; footprint (none) -> LED_SMD:LED_0805_2012Metric
- J2: renamed from J?; footprint (none) -> Connector_PinHeader_2.54mm:PinHeader_1x04_P2.54mm_Vertical
- R39, R40, R41: renamed from R?; footprint (none) -> Resistor_SMD:R_0603_1608Metric
- SW10: renamed from SW?; footprint (none) -> Button_Switch_THT:SW_PUSH_6mm
- TP1, TP2, TP3, TP4, TP5, TP6: renamed from TP?; footprint (none) -> TestPoint:TestPoint_Pad_D2.0mm
Changed lines of the file:
@@
 	10260 4290 10330 4290
 $Comp
-L Switch:SW_Push SW?
+L Switch:SW_Push SW10
 U 1 1 6245B6A5
 P 10000 4680
-F 0 "SW?" H 10000 4555 50  0000 C CNN
+F 0 "SW10" H 10000 4555 50  0000 C CNN
 F 1 "RESET" H 10000 4630 50  0000 C CNN
-F 2 "" H 10000 4880 50  0001 C CNN
+F 2 "Button_Switch_THT:SW_PUSH_6mm" H 10000 4880 50  0001 C CNN
 F 3 "~" H 10000 4880 50  0001 C CNN
 	1    10000 4680
@@
 	10200 4680 10200 4450
 $Comp
-L Device:LED D?
+L Device:LED D1
 U 1 1 624898D2
 P 8400 2550
-F 0 "D?" H 8393 2767 50  0000 C CNN
+F 0 "D1" H 8393 2767 50  0000 C CNN
 F 1 "LED" H 8393 2676 50  0000 C CNN
-F 2 "" H 8400 2550 50  0001 C CNN
+F 2 "LED_SMD:LED_0805_2012Metric" H 8400 2550 50  0001 C CNN
 F 3 "~" H 8400 2550 50  0001 C CNN
 	1    8400 2550
@@
 	7550 2550 8250 2550
 $Comp
-L Device:R R?
+L Device:R R39
 U 1 1 6249085C
 P 8830 2550
-F 0 "R?" V 8623 2550 50  0000 C CNN
+F 0 "R39" V 8623 2550 50  0000 C CNN
 F 1 "R" V 8714 2550 50  0000 C CNN
-F 2 "" V 8760 2550 50  0001 C CNN
+F 2 "Resistor_SMD:R_0603_1608Metric" V 8760 2550 50  0001 C CNN
 F 3 "~" H 8830 2550 50  0001 C CNN
 	1    8830 2550
@@
 $EndComp
 $Comp
-L Device:LED D?
+L Device:LED D3
 U 1 1 624A4D0B
 P 10810 2560
-F 0 "D?" V 10803 2777 50  0000 C CNN
+F 0 "D3" V 10803 2777 50  0000 C CNN
 F 1 "3.3V_LED" V 10720 2760 50  0000 C CNN
-F 2 "" H 10810 2560 50  0001 C CNN
+F 2 "LED_SMD:LED_0805_2012Metric" H 10810 2560 50  0001 C CNN
 F 3 "~" H 10810 2560 50  0001 C CNN
 	1    10810 2560
@@
 $EndComp
 $Comp
-L Device:R R?
+L Device:R R41
 U 1 1 624A4D11
 P 10810 2130
-F 0 "R?" H 10603 2130 50  0000 C CNN
+F 0 "R41" H 10603 2130 50  0000 C CNN
 F 1 "R" H 10694 2130 50  0000 C CNN
-F 2 "" V 10740 2130 50  0001 C CNN
+F 2 "Resistor_SMD:R_0603_1608Metric" V 10740 2130 50  0001 C CNN
 F 3 "~" H 10810 2130 50  0001 C CNN
 	1    10810 2130
@@
 	10810 2710 10810 2880
 $Comp
-L Device:LED D?
+L Device:LED D2
 U 1 1 624BAEF6
 P 10200 2560
-F 0 "D?" V 10239 2442 50  0000 R CNN
+F 0 "D2" V 10239 2442 50  0000 R CNN
 F 1 "5V_LED" V 10130 2910 50  0000 R CNN
-F 2 "" H 10200 2560 50  0001 C CNN
+F 2 "LED_SMD:LED_0805_2012Metric" H 10200 2560 50  0001 C CNN
 F 3 "~" H 10200 2560 50  0001 C CNN
 	1    10200 2560
@@
 $EndComp
 $Comp
-L Device:R R?
+L Device:R R40
 U 1 1 624BAEFC
 P 10200 2130
-F 0 "R?" H 9993 2130 50  0000 C CNN
+F 0 "R40" H 9993 2130 50  0000 C CNN
 F 1 "R" H 10084 2130 50  0000 C CNN
-F 2 "" V 10130 2130 50  0001 C CNN
+F 2 "Resistor_SMD:R_0603_1608Metric" V 10130 2130 50  0001 C CNN
 F 3 "~" H 10200 2130 50  0001 C CNN
 	1    10200 2130
@@
 $EndComp
 $Comp
-L Connector:Conn_01x04_Male J?
+L Connector:Conn_01x04_Male J2
 U 1 1 624CDCE4
 P 4500 6800
-F 0 "J?" H 4270 6790 50  0000 C CNN
+F 0 "J2" H 4270 6790 50  0000 C CNN
 F 1 "SWD" H 4240 6690 50  0000 C CNN
-F 2 "" H 4500 6800 50  0001 C CNN
+F 2 "Connector_PinHeader_2.54mm:PinHeader_1x04_P2.54mm_Vertical" H 4500 6800 50  0001 C CNN
 F 3 "~" H 4500 6800 50  0001 C CNN
 	1    4500 6800
@@
 $EndComp
 $Comp
-L Connector:TestPoint TP?
+L Connector:TestPoint TP1
 U 1 1 624D6BA0
 P 2430 3590
-F 0 "TP?" H 2500 3730 50  0000 L CNN
+F 0 "TP1" H 2500 3730 50  0000 L CNN
 F 1 "D-" H 2660 3730 50  0000 L CNN
-F 2 "" H 2630 3590 50  0001 C CNN
+F 2 "TestPoint:TestPoint_Pad_D2.0mm" H 2630 3590 50  0001 C CNN
 F 3 "~" H 2630 3590 50  0001 C CNN
 	1    2430 3590
@@
 $EndComp
 $Comp
-L Connector:TestPoint TP?
+L Connector:TestPoint TP2
 U 1 1 624D7D3E
 P 2430 3790
-F 0 "TP?" H 2500 3930 50  0000 L CNN
+F 0 "TP2" H 2500 3930 50  0000 L CNN
 F 1 "D+" H 2660 3930 50  0000 L CNN
-F 2 "" H 2630 3790 50  0001 C CNN
+F 2 "TestPoint:TestPoint_Pad_D2.0mm" H 2630 3790 50  0001 C CNN
 F 3 "~" H 2630 3790 50  0001 C CNN
 	1    2430 3790
@@
 	2700 6150 3150 6150
 $Comp
-L Connector:TestPoint TP?
+L Connector:TestPoint TP4
 U 1 1 624E5799
 P 3050 6110
-F 0 "TP?" H 3120 6250 50  0000 L CNN
+F 0 "TP4" H 3120 6250 50  0000 L CNN
 F 1 "SCL" H 3280 6250 50  0000 L CNN
-F 2 "" H 3250 6110 50  0001 C CNN
+F 2 "TestPoint:TestPoint_Pad_D2.0mm" H 3250 6110 50  0001 C CNN
 F 3 "~" H 3250 6110 50  0001 C CNN
 	1    3050 6110
@@
 $EndComp
 $Comp
-L Connector:TestPoint TP?
+L Connector:TestPoint TP3
 U 1 1 624E5A5C
 P 2950 6020
-F 0 "TP?" H 3020 6160 50  0000 L CNN
+F 0 "TP3" H 3020 6160 50  0000 L CNN
 F 1 "SDA" H 3180 6160 50  0000 L CNN
-F 2 "" H 3150 6020 50  0001 C CNN
+F 2 "TestPoint:TestPoint_Pad_D2.0mm" H 3150 6020 50  0001 C CNN
 F 3 "~" H 3150 6020 50  0001 C CNN
 	1    2950 6020
@@
 Connection ~ 2950 6350
 $Comp
-L Connector:TestPoint TP?
+L Connector:TestPoint TP6
 U 1 1 624F3AA9
 P 10810 890
-F 0 "TP?" H 10880 1030 50  0000 L CNN
+F 0 "TP6" H 10880 1030 50  0000 L CNN
 F 1 "3.3V" H 11040 1030 50  0000 L CNN
-F 2 "" H 11010 890 50  0001 C CNN
+F 2 "TestPoint:TestPoint_Pad_D2.0mm" H 11010 890 50  0001 C CNN
 F 3 "~" H 11010 890 50  0001 C CNN
 	1    10810 890
@@
 $EndComp
 $Comp
-L Connector:TestPoint TP?
+L Connector:TestPoint TP5
 U 1 1 624FC023
 P 6000 6580
-F 0 "TP?" H 6070 6720 50  0000 L CNN
+F 0 "TP5" H 6070 6720 50  0000 L CNN
 F 1 "SCL" H 6230 6720 50  0000 L CNN
-F 2 "" H 6200 6580 50  0001 C CNN
+F 2 "TestPoint:TestPoint_Pad_D2.0mm" H 6200 6580 50  0001 C CNN
 F 3 "~" H 6200 6580 50  0001 C CNN
 	1    6000 6580
@@
 $EndComp
 $Comp
-L power:GND #PWR?
+L power:GND #PWR0110
 U 1 1 624FC62E
 P 6000 6640
-F 0 "#PWR?" H 6000 6390 50  0001 C CNN
+F 0 "#PWR0110" H 6000 6390 50  0001 C CNN
 F 1 "GND" H 6005 6467 50  0000 C CNN
 F 2 "" H 6000 6640 50  0001 C CNN
