File: pcb/stream_deck_hardware.kicad_pcb (KiCad board)
At the start: 2 copper layers, 70 x 100 mm, 134 parts, among them J1 USB_C_Receptacle_USB2.0, J10 GND, J11 +5V, J12 DATA, J13 GND, J6 ENC A, J7 ENC B, J8 BUTTON, J9 GND, SW1 SW_Push1, SW2 SW_Push2, SW3 SW_Push3, SW4 SW_Push, SW5 SW_Push, SW6 SW_Push, SW7 SW_Push, SW8 SW_Push, SW9 SW_Push, U1 LF33_TO252, U2 STM32F401RCTx, U3 74LVC1G332, U4 AT24CS02-STUM, U5 AT24CS02-STUM, Y1 Crystal_Small

Commit message: update
Parts:
- moved D+ 3.15 mm to (95.4, 57.5)
- moved D- 3.10 mm to (98.6, 57.5)
- moved C20 1.50 mm to (87.1, 140.0)
- moved R21 1.50 mm to (87.1, 142.0)
- moved R25 1.50 mm to (91.1, 140.0)
Routing:
- net +5V: track 143.0 -> 204.0 mm
- net +3V3: track 32.4 -> 41.1 mm, vias 0 -> 16
- net USB_D-: track 27.1 -> 18.7 mm, vias 2 -> 0
- net USB_D+: track 27.8 -> 21.0 mm
- net Net-(D11-Pad2): track 44.7 -> 45.5 mm
- added copper zone on In1.Cu, net +3V3
- added copper zone on F.Cu, net GND
Other:
- copper layers 2 -> 4

Commit message: commit
Parts:
- moved 3V3 9.40 mm to (118.6, 75.7)
Routing:
- net +3V3: track 41.1 -> 45.1 mm, vias 16 -> 38
- net Button_7: track 0.00 -> 1.38 mm, vias 0 -> 1
- net BOOT0: track 0.00 -> 1.08 mm, vias 0 -> 1
